File: pcb/BioZ-Muscle-Monitor.kicad_pcb (KiCad board)
At the start: 6 copper layers, 62 x 44 mm, 92 parts, among them IC1 CY15V108QI, J1 S4B-PH-K-S, J2 62201021121 SWD, J7 S2B-PH-SM4-TB BATT, J8 S2B-PH-SM4-TB SW, P1 S3B-PH-SM4-TB, SW1 52-03-80 (panel), U1 MAX30009ENA+, U10 ADPL40502-1.8 A, U14 ADPL40502-1.8 D, U2 SN74LVC1G14, U5 nRF54L15-QFAA, U7 MAX77827BEFD+T, U8 BQ24073RGT, U9 103AT-2 (on cell), Y1 32.768kHz ABS06, Y2 32MHz ABM10

Commit message: PCB: pad-stub exception with real measurement, SPI_SCK reroute, root cause found
Pad-stub exception applied properly, not as originally proposed: measured
each of the 7 cases individually rather than trusting the prior session's
assumption. V2P5's "stub" was actually 2.4mm with only the first 0.6mm
pinched -- split into a narrow tip plus full-width run rather than
excusing the whole thing. Three of seven needed a floor of 0.150mm, not
the pad width, because they were tighter than their own pad. Six scoped
rule areas (3.6mm2 total) added, each proven not to leak with a control
test. IR-drop verified with real numbers: worst case 193uV on a 2.5V
rail (0.008%), closing the gap the prior session had left unverified.

SPI_SCK: found to be looping 14.8mm of copper (an old autorouter detour)
to span a 2.6mm distance. Re-laid direct at 4 segments / 2.9mm, freeing
the corridor and letting 3 more V2P5F segments widen for free.

Root cause found for why the board has been stuck near 45 unconnected for
three sessions: 44 of 74 remaining net endpoints physically cannot emit
their brief-mandated trace width at all, because U5's 0.4mm-pitch QFN
pads (0.200mm), U8's pads (0.250mm, narrower than the 0.254mm SIGNAL
floor by 4 microns), and 0201 caps (0.420mm) are all narrower than the
net class's stated minimum. This is the same rule-scope pattern already
found and fixed four times this project, now understood to be the
dominant cause rather than isolated cases.

Session total: 14 -> 1 violation, 45 -> 43 unconnected.

Co-Authored-By: Claude Sonnet 5 <noreply@anthropic.com>
Routing:
- net V2P5: track 10.9 -> 48.5 mm, vias 0 -> 4
- net SPI_SCK: track 31.3 -> 19.8 mm
